File: KiCAD/chipcon.sch (KiCad schematic (older format))
At the start: 37 parts, among them CON1 BARREL_JACK, J1 audio_out, J2 video out, P1 SD card, P2 ICSP, SW1 reset, SW2 power, U1 ATMEGA328-PU, U2 23LC512, U3 LT1117-3,3, X1 16Mhz, k1 KEYPAD

Commit message: modification vm et autre
Parts:
- removed RV1: 10K, ~, symbol POT
- removed k1: KEYPAD, ~, symbol KEYPAD
- added J2: DB9, symbol DB9
- renumbered J2 to J3
Connections:
- net 3,3V: now also J2.7 (P7)
- net GND: now also J2.8 (P8)
- net KP1: no longer names the net of U1.2 (PD0/PCINT16/RXD)
- net KP2: no longer names the net of U1.4 (PD2/PCINT18/INT0)
- net KP3: no longer names the net of U1.5 (PD3/PCINT19/OC2B/INT1)
- net KP4: no longer names the net of U1.11 (PD5/PCINT21/OC0B/T1)
- net KP5 renamed FIRE
- net FIRE: now also J2.6 (P6)
- net KP6 renamed RIGHT
- net RIGHT: now also J2.4
- net KP7 renamed LEFT
- net LEFT: now also J2.3
- net KP8 renamed DOWN
- net DOWN: now also J2.2
- net speed renamed UP
- net UP: now also J2.1
Other:
- note added: "joystick\nAtari 2600"
- note removed: "1) 1-5 9) 3-7\n2) 1-6 A) 1-8\n3) 1-7 B) 2-8\n4) 2-5 C) 3-8\n5) 2-6 D) 4-8\n6) 2-7 #) 4-7\n7) 3-5 *) 4-5\n8) 3-6 0) 4-6"
- note removed: "inputs"
- note removed: "matrice clavier\n"
- note removed: "outputs"

Commit message: travail sur tvout.c
Parts:
- added C1, C6: 100nF, ~, symbol C
- added Q1: 2N7000, ~, symbol MOSFET_N
- added R2: 1K, ~, symbol R
- added R3: 200K, ~, symbol R
- renumbered C8 to C10, C9 to C11, C10 to C12, C11 to C13, C1 to C2, C2 to C3, C3 to C4, C4 to C5, C5 to C7, C6 to C8, C7 to C9, P2 to P1, P1 to P2, R8 to R10, R9 to R11, R10 to R12, R2 to R4, R3 to R5, R4 to R6, R5 to R7, R6 to R8, R7 to R9
Connections:
- net GND: now also C1.1, C6.1, R2.2
- net audio out: now also Q1.D; no longer R1.2
- net Env.: now reaches U1.2 (PD0/PCINT16/RXD)
- net Env.: now also R3.2
- new net: Q1.S, R1.2, R2.1
- new net: C1.2, R3.1
Other:
- note added: "CHIPCON V2\n"
- note added: "Jacques Deschênes\nCopyright 2014,2015\nlicence CC-SA-BY V3"
- note removed: "CHIPCON\n"
- moved on the sheet: C10, C11, C12, C13, C2, C3, C4, C5, C7, C8, C9, CON1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
